File: pcb/jak.kicad_sch (KiCad schematic)
At the start: 92 parts, among them SW1 SW_Push, SW10 SW_Push, SW10_r1 SW_Push, SW11 SW_Push, SW11_r1 SW_Push, SW12 SW_Push, SW12_r1 SW_Push, SW13 SW_Push, SW13_r1 SW_Push, SW14 SW_Push, SW14_r1 SW_Push, SW15 SW_Push, SW15_r1 SW_Push, SW16 SW_Push, SW16_r1 SW_Push, SW17 SW_Push, SW17_r1 SW_Push, SW18 SW_Push, SW18_r1 SW_Push, SW1_r1 SW_Push, SW2 SW_Push, SW2_r1 SW_Push, SW3 SW_Push, SW3_r1 SW_Push, SW4 SW_Push, SW4_r1 SW_Push, SW5 SW_Push, SW5_r1 SW_Push, SW6 SW_Push, SW6_r1 SW_Push, SW7 SW_Push, SW7_r1 SW_Push, SW8 SW_Push, SW8_r1 SW_Push, SW9 SW_Push, SW9_r1 SW_Push

Commit message: tt
Parts:
- jst1, jst2, jst_r1, jst_r2: footprint project:2-pin-jst -> jak:2-pin-jst
Changed lines of the file:
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@@
 			)
 		)
-		(property "Footprint" "project:2-pin-jst"
+		(property "Footprint" "jak:2-pin-jst"
 			(at 167.64 152.4 0)
 			(effects
@@
 		(fields_autoplaced yes)
 		(property "Reference" "controller1"
-			(at 38.1 15.24 0)
+			(at 38.1 12.7 0)
 			(effects
 				(font
@@
 		)
 		(property "Value" "ProMicro"
-			(at 38.1 17.78 0)
+			(at 38.1 15.24 0)
 			(effects
 				(font
@@
 		)
 		(property "Footprint" "kbd:ProMicro"
-			(at 40.64 63.5 0)
+			(at 38.1 17.78 0)
 			(effects
 				(font
 					(size 1.524 1.524)
 				)
-				(hide yes)
 			)
 		)
@@
 		(fields_autoplaced yes)
 		(property "Reference" "controller_r1"
-			(at 256.54 13.97 0)
+			(at 256.54 11.43 0)
 			(effects
 				(font
@@
 		)
 		(property "Value" "ProMicro"
-			(at 256.54 16.51 0)
+			(at 256.54 13.97 0)
 			(effects
 				(font
@@
 		)
 		(property "Footprint" "kbd:ProMicro"
-			(at 259.08 62.23 0)
+			(at 256.54 16.51 0)
 			(effects
 				(font
 					(size 1.524 1.524)
 				)
-				(hide yes)
 			)
 		)
@@
 			)
 		)
-		(property "Footprint" "project:2-pin-jst"
+		(property "Footprint" "jak:2-pin-jst"
 			(at 67.31 175.26 0)
 			(effects
@@
 			)
 		)
-		(property "Footprint" "project:2-pin-jst"
+		(property "Footprint" "jak:2-pin-jst"
 			(at 167.64 163.83 0)
 			(effects
@@
 			)
 		)
-		(property "Footprint" "project:2-pin-jst"
+		(property "Footprint" "jak:2-pin-jst"
 			(at 67.31 162.56 0)
 			(effects

Commit message: In the process of transitioning the board to use the SEEED XIAO instead of a pro micro
Parts:
- removed RSW1, RSW2: SW_Push, kbd:ResetSW, symbol Switch:SW_Push
- removed controller1, controller_r1: ProMicro, kbd:ProMicro, symbol kbd:ProMicro
- removed jst2, jst_r1, jst_r2: Conn_01x02, jak:2-pin-jst, symbol Connector_Generic:Conn_01x02
- added RES1, RES_r1: PTS526 SM15 SMTR2 LFS, footprints:SON4_PTS526 SM15 SMTR2 LFS_CNK, symbol 2026-01-19_20-43-58:PTS526_SM15_SMTR2_LFS
- added controller1, controller_r1: XIAO-nRF52840-SMD, jak:XIAO-nRF52840-SMD-underside, symbol Seeed_Studio_XIAO_Series:XIAO-nRF52840-SMD
- added jst_r1: S2B-PH-K-S_LF__SN_, S2B-PH-K-S_LF__SN_:JST_S2B-PH-K-S_LF__SN_, symbol S2B-PH-K-S_LF__SN_:S2B-PH-K-S_LF__SN_
- jst1: footprint jak:2-pin-jst -> S2B-PH-K-S_LF__SN_:JST_S2B-PH-K-S_LF__SN_; symbol Connector_Generic:Conn_01x02 -> S2B-PH-K-S_LF__SN_:S2B-PH-K-S_LF__SN_; AVAILABILITY (none) -> Unavailable; Availability (none) -> In Stock; Check_prices (none) -> https://www.snapeda.com/parts/S2B-PH-K-S(LF)(SN)/JST/view-p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; DESCRIPTION (none) -> Connector Header Through Hole, Right Angle 2 position; Description_1 (none) -> Connector Header Through Hole, Right Angle 2 position; MAXIMUM_PACKAGE_HEIGHT (none) -> 4.8mm; MF (none) -> JST Sales America Inc.; MP (none) -> S2B-PH-K-S(LF)(SN); PACKAGE (none) -> None; PRICE (none) -> None; Package (none) -> NON STANDARD-2 J.S.T.; Price (none) -> None; SnapEDA_Link (none) -> https://www.snapeda.com/parts/S2B-PH-K-S(LF)(SN)/JST/view-p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
- power1, power_r1: footprint Kicad-Footprints:SPDT_C128955 -> Button_Switch_SMD:SW_SPDT_PCM12
Connections:
- net GND: now also RES1.3, RES1.4, controller1.13 (GND), controller1.16 (GND), controller1.22 (GND)
- net GND_r: now also RES_r1.1, RES_r1.2, controller_r1.13 (GND), controller_r1.16 (GND), controller_r1.22 (GND), jst_r1.1
- net VCC: now also controller1.12 (3V3)
- net VCC_r: now also controller_r1.12 (3V3)
- net battery+_r: now also power_r1.1 (A), jst_r1.2; no longer power_r1.3 (C)
- net col0: now also controller1.6 (P0.05_A5_D5_SCL)
- net col0_r: now also controller_r1.6 (P0.05_A5_D5_SCL)
- net col1: now also controller1.5 (P0.04_A4_D4_SDA)
- net col1_r: now also controller_r1.5 (P0.04_A4_D4_SDA)
- net col2: now also controller1.9 (P1.13_D8_SCK)
- net col2_r: now also controller_r1.9 (P1.13_D8_SCK)
- net col3: now also controller1.10 (P1.14_D9_MISO)
- net col3_r: now also controller_r1.10 (P1.14_D9_MISO)
- net col4: now also controller1.11 (P1.15_D10_MOSI)
- net col4_r: now also controller_r1.11 (P1.15_D10_MOSI)
- net reset: now also RES1.1, RES1.2, controller1.21 (RESET)
- net reset_r: now also RES_r1.3, RES_r1.4, controller_r1.21 (RESET)
- net row0: now also controller1.1 (P0.02_A0_D0)
- net row0_r: now also controller_r1.1 (P0.02_A0_D0)
- net row1: now also controller1.2 (P0.03_A1_D1)
- net row1_r: now also controller_r1.2 (P0.03_A1_D1)
- net row2: now also controller1.3 (P0.28_A2_D2)
- net row2_r: now also controller_r1.3 (P0.28_A2_D2)
- net row3: now also controller1.4 (P0.29_A3_D3)
- net row3_r: now also controller_r1.4 (P0.29_A3_D3)
- net split_comms+: now also controller1.7 (P1.11_D6_TX)
- net split_comms+_r: now also controller_r1.8 (P1.12_D7_RX)
- net split_comms-: now also controller1.8 (P1.12_D7_RX)
- net split_comms-_r: now also controller_r1.7 (P1.11_D6_TX)
- net raw renamed battery_switched
- net battery_switched: now also controller1.15 (BAT)
- net raw_r renamed battery_switched_r
- net battery_switched_r: now also controller_r1.15 (BAT)
- no-connect marks 24 -> 20
Other:
- moved on the sheet: D1, D10, D11, D12, D13, D14, D15, D16, D17, D18, D19, D2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
